File: CurrentMonitor.sch (EAGLE design)
At the start: 75 parts, among them IC1 MEGA8-AI, IC2 INA138, IC3 INA138, IC4 LF33CV, J1 AVR_SPI_PRG_6OFFSET_PADS, Q1 10MHz, Q2 IRLZ34N, Q3 IRLZ34N, Q4 IRLZ34N, Q6 BC847, Q7 IRF9530, Q8 IRF9530, Q9 BC847, X1 MSTBA2, X2 MSTBA2, X3 MSTBA2, X5 MSTBA2

Commit message: Few fixes (forgot to commit, forgot what I have changed) ;)
Parts:
- removed C13: 1µ, rcl:CPOL-EUB
- added C150, C200: 150µ/25V, rcl:CPOL-EUF
- added C201: 1µ/25V, rcl:CPOL-EUB
- added C202: 100n, resistor:C-EUC0805
- added C3, C4: (no value), rcl:CPOL-EUE3.5-8
- added IC5: DS18S20, 1wire:DS18S20
- added IC6: 7805TV, linear:7805TV
- added J2, J3: 22-27-2051-05, con-molex:22-27-2051-05
- added J4: 22-27-2021-02, con-molex:22-27-2021-02
- added Q10: BS170, transistor-small-signal:BS170
- added R100, R102: 0.1, resistor:R-EU_R1206
- added R101, R103: 0.005, resistor:R-EU_R2512
- added R200: 200, rcl:R-EU_R0805
- added SV1: (no value), con-ml:ML14
- added U$13, U$14: LITTLEFUSE-178.6164, PudenzCarFuseFLR:LITTLEFUSE-178.6164
- added U$3: TINY2313-*S*, avr-7:TINY2313-*S*
- added X4: 231-432/001-000, con-wago_5.0mm:231-432/001-000
- added X6: 231-433/001-000, con-wago_5.0mm:231-433/001-000
- added Y1: (no value), SparkFun:CRYSTALHC49US
- C10: value 100n -> (none); device resistor:C-EUC0805 -> rcl:C-EUC0805
- C11, C12: value 100µ -> (none); device rcl:CPOL-EUF -> resistor:C-EUC0805
- C151: value 1µ -> 1µ/25V
- C20: device rcl:CPOL-EUA/3216-18R -> rcl:CPOL-EUA
- D3: device diode:1N4004 -> gm-diodes:DO41.3
- JP1: value (none) -> AVR-ISP-6VERT; device pinhead:PINHD-1X6 -> avr-7:AVR-ISP-6VERT
- Q5: value (none) -> BS170; device crystal:CRYSTALHC49S -> transistor-small-signal:BS170
- R1, R10, R11, R12, R13, R18, R19, R23, R25, R26, R27, R28, R3, R6, R8, R9: device rcl:R-EU_R1206 -> rcl:R-EU_R0805
- R14: device resistor:R-EU_R1206 -> rcl:R-EU_R0805
- R15, R16: device resistor:R-EU_R1206 -> resistor:R-EU_R0805
- R17: value 200 -> (none); device resistor:R-EU_R1206 -> pot:TRIM_EU-PT10
- R2: value 0.1 -> (none); device resistor:R-EU_R1206 -> rcl:R-EU_R0805
- R20: value 10k -> (none); device rcl:R-EU_R1206 -> pot:TRIM_EU-PT10
- R21: value 10k -> (none); device rcl:R-EU_R1206 -> rcl:R-EU_R0805
- R22, R24: device rcl:R-EU_R1206 -> resistor:R-EU_R0805
- R4, R7: device rcl:R-TRIMM64P -> rcl:R-TRIMM64W
- R5: value 0.1 -> (none); device resistor:R-EU_R1206 -> resistor:R-EU_R0805
- X1, X2, X3: value MSTBA2 -> 231-432/001-000; device con-phoenix-508:MSTBA2 -> con-wago_5.0mm:231-432/001-000
- X5: value MSTBA2 -> 231-433/001-000; device con-phoenix-508:MSTBA2 -> con-wago_5.0mm:231-433/001-000
- renumbered C14 to C151
Connections:
- new net +3V3_2: C10.1, IC5P.VDD, J2-2.S, JP2.1, R2.2, R5.2, U$3.VCC, X6.P3
- new net +5V_2: C4.+, IC6.VO, Q10.D, R20.E, SV1.1
- new net BAT+CON: U$14.2, X2.P1
- new net BAT+_2: J2-3.S, Q5.D
- new net BGEN: Q10.G, U$3.(OC1B)PB4
- new net DB4: SV1.11, U$3.(TXD)PD1
- new net DB5: SV1.12, U$3.(INT0)PD2
- new net DB6: SV1.13, U$3.(INT1)PD3
- new net DB7: SV1.14, U$3.(T0)PD4
- new net DISPLAYEN: Q5.G, U$3.(OC1A)PB3
- new net E: SV1.6, U$3.(T1)PD5
- new net FROM_CELL_CON: U$13.2, X1.P1
- new net GND_2: C10.2, C11.1, C12.1, C3.-, C4.-, IC5P.GND, IC6.GND, J2-1.S, J4-1.S, JP1.6, JP2.4, R20.A, SV1.2, U$3.GND, X6.P1
- new net N$15: R17.S, R21.1
- new net N$19: JP2.2, R5.1, U$3.(ICP)PD6
- new net N$24: J4-2.S, R21.2
- new net N$27: JP1.5, R2.1, U$3.PA2(/RESET)
- new net N$28: Q10.S, R17.E
- new net N$30: C11.2, U$3.PA1(XTAL2), Y1.2
- new net N$31: C12.2, U$3.PA0(XTAL1), Y1.1
- new net N$33: C3.+, IC6.VI, Q5.S
- new net N$35: U$3.(OC0A)PB2
- new net N$7: JP1.1, U$3.(MISO)PB6
- new net OW: IC5_1W.1W, U$3.(RXD)PD0, X6.P2
- new net R/W: SV1.5, U$3.(AIN0)PB0
- new net RS: R20.S, SV1.4, U$3.(AIN1)PB1
- new net SCL2: J2-5.S, JP1.3, U$3.(UCSK)PB7
- new net SDA2: J2-4.S, JP1.4, U$3.(MOSI)PB5
- new net V0: SV1.3
- net +3V3: now also J3-2.S; no longer JP1.3, JP1.4, R20.1, R21.1
- net BAT+: now also J3-3.S, R102.2, R103.1, U$14.1; no longer JP1.5, JP1.6, R5.2, X2-1.1
- net CELL_TO_CONTROLLER: now also C150.+, R100.2, R101.1; no longer C12.+, R2.2
- net CONTROLLER_TO_BAT: now also C200.+, C201.+, R102.1, R103.2, R200.2; no longer C11.+, C13.+, R17.2, R5.1
- net FROM_CELL: now also R100.1, R101.2, U$13.1; no longer R2.1, X1-1.1
- net GND: now also C150.-, C200.-, C201.-, J3-1.S, X1.P2, X2.P2, X3.P1, X4.P1, X5.P1; no longer C11.-, C12.-, C13.-, JP1.1, JP1.2, X1-2.1, X2-2.1, X3-2.1, X5-2.1
- net N$16: now also X3.P2; no longer X3-1.1
- net N$17: now also C202.1, R200.1; no longer C10.1, R17.1
- net N$25: now also X4.P2; no longer X5-1.1
- net RXD: no longer JP2.3
- net SCL: now also J3-5.S, X5.P2; no longer JP2.2, R21.2
- net SDA: now also J3-4.S, X5.P3; no longer JP2.1, R20.2
- net TXD: no longer JP2.4
- net VS: now also C202.2; no longer C10.2
- net XTAL1: no longer Q5.2
- net XTAL2: no longer Q5.1
Other:
- note added: "0..25V 0..10A (fit R101)"
- note added: "0..25V 0..10A (fit R103)"
- note added: "0..25V 0..2A (fit R100)"
- note added: "0..25V 0..2A (fit R102)"
- note added: "C150 needs to have an ESR of 0.1 Ohm or lower"
- note added: "C200 needs to have an ESR of 0.1 Ohm or lower"
- note added: "Design Notes: - The design is based on the freechargecontroller.org design, which in turn is based on Tim Noland's design - Full current/voltage monitoring for both cell and circuit - Load On/Off via P-Channel Mosfet - Provides 3.3V output (0.8A maximum) to power other 3.3V loads, also switchable via P-Channel Mosfet - Can be built in different variants: 2A or 5A - Microcontroller acts as a I²C S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"
- note removed: "0..25V 0..2A"
- note removed: "I²C Pullups"
